File: FOC_INVERTER/FOC_INVERTER.kicad_sch (KiCad schematic)
At the start: 0 parts

Commit message: LAST
Parts:
- added C1, C17, C18, C2, C4, C5, C6, C7, C8: 100nF, Capacitor_THT:C_Disc_D5.0mm_W2.5mm_P2.50mm, symbol Device:C
- added C10, C9: 100uF, Capacitor_THT:CP_Radial_D7.5mm_P2.50mm, symbol Device:C_Polarized
- added C11, C12, C13, C14, C15, C16: 100pF, Capacitor_SMD:C_0603_1608Metric, symbol Device:C
- added C19: 470pF, Capacitor_SMD:C_0603_1608Metric, symbol Device:C
- added C20: 200nF, Capacitor_THT:C_Disc_D5.0mm_W2.5mm_P2.50mm, symbol Device:C
- added C3: C, Capacitor_THT:C_Disc_D5.0mm_W2.5mm_P2.50mm, symbol Device:C
- added D1, D2, D3, D4, D5, D6: 1N4148, Diode_THT:D_DO-35_SOD27_P7.62mm_Horizontal, symbol Diode:1N4148
- added EN1: BLUE - 3MM, LED_THT:LED_D3.0mm_IRBlack, symbol LED:IR204A
- added FAULT1: RED - 3MM, LED_THT:LED_D3.0mm_IRBlack, symbol LED:IR204A
- added J1: Conn_01x10_Pin, Connector_JST:JST_XH_S10B-XH-A-1_1x10_P2.50mm_Horizontal, symbol Connector:Conn_01x10_Pin
- added J2: Conn_01x03_Pin, Connector_Phoenix_MC_HighVoltage:PhoenixContact_MCV_1,5_3-G-5.08_1x03_P5.08mm_Vertical, symbol Connector:Conn_01x03_Pin
- added R1, R10, R12, R20, R22, R2_T1, R4, R6, R8: 1K, Resistor_THT:R_Axial_DIN0204_L3.6mm_D1.6mm_P7.62mm_Horizontal, symbol Device:R
- added R11, R19, R2, R3, R9: 200, Resistor_THT:R_Axial_DIN0204_L3.6mm_D1.6mm_P7.62mm_Horizontal, symbol Device:R
- added R13, R14, R15, R16, R17, R18: 200, Resistor_SMD:R_0805_2012Metric, symbol Device:R
- added R1_T1: 10k Ω, Potentiometer_THT:Potentiometer_Bourns_3386P_Vertical, symbol Device:R_Potentiometer_Trim
- added R21: 1.3K, Resistor_THT:R_Axial_DIN0204_L3.6mm_D1.6mm_P7.62mm_Horizontal, symbol Device:R
- added R23, R24, R25: 3KΩ, Resistor_THT:R_Axial_DIN0204_L3.6mm_D1.6mm_P7.62mm_Horizontal, symbol Device:R
- added R26: 0.11 Ω, Resistor_THT:R_Axial_Power_L38.0mm_W6.4mm_P45.72mm, symbol Device:R
- added R27: 1kΩ, Resistor_SMD:R_0805_2012Metric, symbol Device:R
- added R28: 200KΩ, Resistor_SMD:R_0805_2012Metric, symbol Device:R
- added R29, R31, R33, R35, R37, R39: 10Ω, Resistor_SMD:R_1206_3216Metric, symbol Device:R
- added R30, R32, R34, R36, R38, R40: 17Ω, Resistor_SMD:R_1206_3216Metric, symbol Device:R
- added R5, R7: R, Resistor_THT:R_Axial_DIN0204_L3.6mm_D1.6mm_P7.62mm_Horizontal, symbol Device:R
- added STP20NM60FP1, STP20NM60FP2, STP20NM60FP3, STP20NM60FP4, STP20NM60FP5, STP20NM60FP6: STP20NM60FP, Package_TO_SOT_THT:TO-220-3_Vertical, symbol Driver_FET_Custom:STP20NM60FP
- added U1: IR2136S, Package_SO:SOIC-28W_7.5x17.9mm_P1.27mm, symbol Driver_FET_Custom:IR2136S
- added U10, U9: PC817, Package_DIP:DIP-4_W7.62mm, symbol Isolator:PC817
- added U2, U4, U5, U6, U7, U8: 6N137, Package_DIP:DIP-8_W7.62mm, symbol Isolator:6N137
- added U3: LM7805_TO220, Package_TO_SOT_THT:TO-220-3_Vertical, symbol Regulator_Linear:LM7805_TO220
- added VCC1: GREEN - 3MM, LED_THT:LED_D3.0mm_IRBlack, symbol LED:IR204A
Connections:
- new net: R25.2, VCC1.1 (K)
- new net: D3.1 (K), R33.2
- new net: C16.1, R13.2, U1.2 (~{HIN1})
- new net: R7.2, U6.2 (A)
- new net: C20.1, R28.2
- new net: D6.1 (K), R39.2
- new net: D5.2 (A), R38.2, STP20NM60FP2.1 (G)
- new net: D6.2 (A), R40.2, STP20NM60FP4.1 (G)
- new net: STP20NM60FP1.2 (D), STP20NM60FP4.3 (S)
- new net: D4.1 (K), R35.2
- new net: C13.1, R16.2, U1.5 (~{LIN1})
- new net: FAULT1.1 (K), R23.2
- new net: D4.2 (A), R36.2, STP20NM60FP5.1 (G)
- new net: C12.1, R17.2, U1.6 (~{LIN2})
- new net: R21.2, U9.1
- new net: D2.1 (K), R31.2
- new net: D5.1 (K), R37.2
- new net: C14.1, R15.2, U1.4 (~{HIN3})
- new net: R11.2, U8.2 (A)
- new net: STP20NM60FP2.2 (D), STP20NM60FP5.3 (S)
- new net: STP20NM60FP1.3 (S), STP20NM60FP2.3 (S), STP20NM60FP3.3 (S)
- new net: D2.2 (A), R32.2, STP20NM60FP3.1 (G)
- new net: R2.2, U2.2 (A)
- new net: R19.2, U10.1
- new net: C15.1, R14.2, U1.3 (~{HIN2})
- new net: D3.2 (A), R34.2, STP20NM60FP6.1 (G)
- new net: R5.2, U5.2 (A)
- new net: STP20NM60FP3.2 (D), STP20NM60FP6.3 (S)
- new net: C11.1, R18.2, U1.7 (~{LIN3})
- new net: R27.2, U1.9 (ITRIP)
- new net: R9.2, U7.2 (A)
- new net: EN1.1 (K), R24.2
- new net: D1.1 (K), R29.2
- new net: D1.2 (A), R30.2, STP20NM60FP1.1 (G)
- new net: R3.2, U4.2 (A)
- new net +15V: C7.1, C9.1, FAULT1.2 (A), R28.1, U1.1 (VCC), U3.1 (VI), VCC1.2 (A)
- new net +5V: C1.1, C10.1, C2.1, C3.1, C4.1, C5.1, C6.1, C8.1, R1.1, R10.1, R12.1, R20.2, R22.2, R4.1, R6.1, R8.1, U2.7 (EN), U2.8 (VCC), U3.3 (VO), U4.7 (EN), U4.8 (VCC), U5.7 (EN), U5.8 (VCC), U6.7 (EN), U6.8 (VCC), U7.7 (EN), U7.8 (VCC), U8.7 (EN), U8.8 (VCC)
- new net +VDC: STP20NM60FP4.2 (D), STP20NM60FP5.2 (D), STP20NM60FP6.2 (D)
- new net COM: R1_T1.3, R26.2, U1.13 (COM)
- new net EN: C17.1, EN1.2 (A), R20.1, U1.10 (EN), U10.4
- new net EN_MCU: J1.3 (Pin_3), R19.1
- new net FAULT: R21.1, R23.1, U1.8 (~{FAULT})
- new net FAULT_MCU: C18.1, J1.1 (Pin_1), R22.1, U9.4
- new net GND: C1.2, C10.2, C11.2, C12.2, C13.2, C14.2, C15.2, C16.2, C17.2, C18.2, C19.2, C2.2, C20.2, C3.2, C4.2, C5.2, C6.2, C7.2, C8.2, C9.2, R24.1, R25.1, R26.1, R2_T1.1, U1.12 (VSS), U10.3, U2.5 (GND), U3.2 (GND), U4.5 (GND), U5.5 (GND), U6.5 (GND), U7.5 (GND), U8.5 (GND), U9.3
- new net GNDD: J1.10 (Pin_10), U10.2, U2.3 (C), U4.3 (C), U5.3 (C), U6.3 (C), U7.3 (C), U8.3 (C), U9.2
- new net HIN1: R1.2, R13.1, U2.6 (VO)
- new net HIN2: R14.1, R6.2, U5.6 (VO)
- new net HIN3: R10.2, R15.1, U7.6 (VO)
- new net HO1: R39.1, R40.1, U1.27 (HO1)
- new net HO2: R35.1, R36.1, U1.23 (HO2)
- new net HO3: R33.1, R34.1, U1.19 (HO3)
- new net ITRIP: C19.1, R1_T1.1, R27.1, R2_T1.2
- new net LIN1: R16.1, R4.2, U4.6 (VO)
- new net LIN2: R17.1, R8.2, U6.6 (VO)
- new net LIN3: R12.2, R18.1, U8.6 (VO)
- new net LO1: R29.1, R30.1, U1.16 (LO1)
- new net LO2: R37.1, R38.1, U1.15 (LO2)
- new net LO3: R31.1, R32.1, U1.14 (LO3)
- new net OUT_A: J2.3 (Pin_3), U1.26 (VS1)
- new net OUT_B: J2.2 (Pin_2), U1.22 (VS2)
- new net OUT_C: J2.1 (Pin_1), U1.18 (VS3)
- new net PWM_U_H: J1.4 (Pin_4), R2.1
- new net PWM_U_L: J1.7 (Pin_7), R3.1
- new net PWM_V_H: J1.5 (Pin_5), R5.1
- new net PWM_V_L: J1.8 (Pin_8), R7.1
- new net PWM_W_H: J1.6 (Pin_6), R9.1
- new net PWM_W_L: J1.9 (Pin_9)
- new net PWM_W_N: R11.1
- new net RCIN: U1.11 (RCIN)
Other:
- note added: "470pF + 1kΩ ITRIP Filte τ = RC = 1kΩ × 470pF = 470ns t_rise (10-90%) ≈ 1.0μs t_90 (settling) ≈ 1.1μs f_cutoff = 1/(2πRC) = 339kHz"
- note added: "Expected current = 0.2A ▲V=10 v P= 2 watt"
- note added: "For Trip current 2x rated I trip = 8x2= 16A ,Rshunt = 0.11 Ω -> I1+I2=16 -> 0.11 I2 = I1(R1+R2) -> I1 x R2 = 0.5 V 2.52 R2 = R1 + 0.11 if R2 = 1kΩ then R1 = 2.72kΩ TRIMMER 10KΩ"
- note added: "Gate drive network for STP20NM60FP: - Vdrive = 15 V (from IR2136) - Series gate resistor Rg = 15-22 Ω - Internal MOSFET gate resistance Rint ≈ 1.6 Ω - Total gate charge Qg ≈ 40-50 nC - Target switching ~100 ns → Ig ≈ 0.5-0.7 A - Optional diode for asymmetrical turn-on/off (ON slower, OFF faster) - Purpose: Limit di/dt, reduce ringing/EMI, protect driver, comply with IEC"
- note added: "I1"
- note added: "I2"
- note added: "INPUT RC FILTER (200Ω + 100pF) • f_c = 8MHz, τ = 20ns • Place C adjacent to IC"
- note added: "MCU INPUT RESISTOR Target current 10 mA forward voltafe 1.4 V 15 V, 1360Ω"
- note added: "MCU INPUT RESISTOR Target current 10 mA forward voltafe 1.4 V 3.3V, 190Ω 5.0V, 360Ω"
- note added: "RCIN Acording to the datasheet fault clearing time τ=R×C τ=R×C=200k×200nF= 40 ms"

Commit message: schematic_done_rev_1.1
Parts:
- added C21, C22, C23, C24, C25, C26: 1nF, Capacitor_THT:C_Disc_D5.0mm_W2.5mm_P2.50mm, symbol Device:C
- added C27, C29, C31, C33: 100nF, Capacitor_THT:C_Disc_D5.0mm_W2.5mm_P2.50mm, symbol Device:C
- added C28, C30, C32, C34: 10uF, Capacitor_THT:CP_Radial_D5.0mm_P2.50mm, symbol Device:C_Polarized
- added D7, D8, D9: UF4007, Diode_THT:D_DO-41_SOD81_P10.16mm_Horizontal, symbol Driver_FET_Custom:UF4007
- added R41, R42, R43, R44, R45, R46: 22Ω, Resistor_THT:R_Axial_DIN0204_L3.6mm_D1.6mm_P7.62mm_Horizontal, symbol Device:R
- added R47: 3KΩ, Resistor_THT:R_Axial_DIN0204_L3.6mm_D1.6mm_P7.62mm_Horizontal, symbol Device:R
- added TVS1, TVS2, TVS3, TVS4, TVS5, TVS6: P6KE18CA, Diode_THT:D_DO-15_P12.70mm_Horizontal, symbol Driver_FET_Custom:P6KE18CA
- added VCC_5V1: yellow - 3MM, LED_THT:LED_D3.0mm_IRBlack, symbol LED:IR204A
- R36: value 17Ω -> 10Ω
- R39: value 10Ω -> 17Ω
- R5, R7: value R -> 200
- renumbered VCC1 to VCC_15
Connections:
- net +15V: now also C33.2, C34.2, D7.2 (A), D8.2 (A), D9.2 (A)
- net +5V: now also VCC_5V1.2 (A)
- net +VDC: now also R41.1, R42.1, R46.1
- net COM: now also STP20NM60FP1.3 (S), STP20NM60FP2.3 (S), STP20NM60FP3.3 (S), C23.2, C24.2, C25.2, C33.1, C34.1, TVS1.2, TVS2.2, TVS5.2
- net GND: now also R47.1
- net HO1: now also D6.2 (A), R40.2, STP20NM60FP4.1 (G), TVS6.1; no longer R39.1, R40.1, U1.27 (HO1)
- net HO2: now also D5.2 (A), R39.2, STP20NM60FP5.1 (G), TVS4.1; no longer R35.1, R36.1, U1.23 (HO2)
- net HO3: now also D4.2 (A), R38.2, STP20NM60FP6.1 (G), TVS3.1; no longer R33.1, R34.1, U1.19 (HO3)
- net LO1: now also D1.2 (A), R30.2, STP20NM60FP1.1 (G), TVS5.1; no longer R29.1, R30.1, U1.16 (LO1)
- net LO2: now also D2.2 (A), R32.2, STP20NM60FP2.1 (G), TVS1.1; no longer R37.1, R38.1, U1.15 (LO2)
- net LO3: now also D3.2 (A), R34.2, STP20NM60FP3.1 (G), TVS2.1; no longer R31.1, R32.1, U1.14 (LO3)
- net OUT_A: now also STP20NM60FP1.2 (D), STP20NM60FP4.3 (S), C26.2, C31.2, C32.2, R45.1, TVS6.2
- net OUT_B: now also STP20NM60FP2.2 (D), STP20NM60FP5.3 (S), C21.2, C29.2, C30.2, R44.1, TVS4.2
- net OUT_C: now also STP20NM60FP3.2 (D), STP20NM60FP6.3 (S), C22.2, C27.2, C28.2, R43.1, TVS3.2
- net RCIN: now also C20.1, R28.2
- net at D6.1 (K): now also R37.2; no longer R39.2
- net at D5.1 (K): now also R36.2; no longer R37.2
- net VB3: now reaches U1.20 (VB3)
- net VB3: now also C27.1, C28.1, D9.1 (K)
- net VB2: now reaches U1.24 (VB2)
- net VB2: now also C29.1, C30.1, D7.1 (K)
- net VB1: now reaches U1.28 (VB1)
- net VB1: now also C31.1, C32.1, D8.1 (K)
- new net: C22.1, R42.2
- new net: C25.1, R45.2
- new net: R31.1, R32.1, U1.15 (LO2)
- new net: R37.1, R40.1, U1.27 (HO1)
- new net: C21.1, R41.2
- new net: R47.2, VCC_5V1.1 (K)
- new net: R35.1, R38.1, U1.19 (HO3)
- new net: R33.1, R34.1, U1.14 (LO3)
- new net: R29.1, R30.1, U1.16 (LO1)
- new net: R36.1, R39.1, U1.23 (HO2)
- new net: C26.1, R46.2
- new net: C24.1, R44.2
- new net: C23.1, R43.2
Other:
- note added: "Gate drive network for STP20NM60FP: - Vdrive = 15 V (from IR2136) - Series gate resistor Rg = 15-22 Ω - Internal MOSFET gate resistance Rint ≈ 1.6 Ω - Total gate charge Qg ≈ 40-50 nC - Target switching ~100 ns → Ig ≈ 0.5-0.7 A - Diode for asymmetrical turn-on/off - Purpose: Limit di/dt, reduce ringing/EMI"
- note added: "INPUT RC FILTER (200Ω + 100pF) • f_c = 8MHz, τ = 20ns"
- note added: "V_bus = 170V DC, I_motor = 8A, f_sw = 8kHz (T=125µs) MOSFET: STP20NM60FP (Q_g = 30nC) Driver: IR2136 (V_CC = 15V, V_UVLO = 8.2V, Q_ls = 20nC max) Diode: UF4007 (V_R = 1000V, V_f = 1.1V @ 0.5A, t_rr = 75ns, Q_rr ≈ 20nC) Capacitor: 150nF 100V X7R (ceramic) + 10µF 100V (electrolytic) per phase Resistor: 4.7Ω 0.5W 1206 (R_boot) Protection: SMAJ18CA TVS across C_boot (clamps >18V spikes) Q_total = (Q_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"
- note removed: "Gate drive network for STP20NM60FP: - Vdrive = 15 V (from IR2136) - Series gate resistor Rg = 15-22 Ω - Internal MOSFET gate resistance Rint ≈ 1.6 Ω - Total gate charge Qg ≈ 40-50 nC - Target switching ~100 ns → Ig ≈ 0.5-0.7 A - Optional diode for asymmetrical turn-on/off (ON slower, OFF faster) - Purpose: Limit di/dt, reduce ringing/EMI, protect driver, comply with IEC"
- note removed: "INPUT RC FILTER (200Ω + 100pF) • f_c = 8MHz, τ = 20ns • Place C adjacent to IC"
- moved on the sheet: C10, C7, C8, C9, R1_T1, R2_T1, STP20NM60FP1, U1, U3
