File: FOC_INVERTER/FOC_INVERTER.kicad_pcb (KiCad board)
At the start: 2 copper layers, 120 parts, among them J1 Conn_01x10_Pin, J2 Conn_01x03_Pin, U1 IR2136S, U10 PC817, U2 6N137, U3 LM7805_TO220, U4 6N137, U5 6N137, U6 6N137, U7 6N137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

Commit message: update
Parts:
- added C35: 100nF, Capacitor_THT:C_Disc_D5.0mm_W2.5mm_P2.50mm, F.Cu at (244.0, 80.9)
- added C36: 1uF, Capacitor_THT:CP_Radial_D5.0mm_P2.50mm, F.Cu at (237.5, 82.1)
- added C37: 100nF, Capacitor_THT:C_Disc_D5.0mm_W2.5mm_P2.50mm, F.Cu at (244.0, 84.9)
- added C38: 1uF, Capacitor_THT:CP_Radial_D5.0mm_P2.50mm, F.Cu at (237.5, 88.7)
- added C39: 100nF, Capacitor_THT:C_Disc_D5.0mm_W2.5mm_P2.50mm, F.Cu at (244.0, 89.0)
- added C40: 1uF, Capacitor_THT:CP_Radial_D5.0mm_P2.50mm, F.Cu at (237.5, 95.2)
- added C41: 2.2uF, Capacitor_THT:C_Disc_D5.0mm_W2.5mm_P2.50mm, F.Cu at (251.5, 86.0)
- added C43: 470pF, Capacitor_THT:C_Disc_D5.0mm_W2.5mm_P2.50mm, F.Cu at (244.0, 93.0)
- added U11: ACS712xLCTR-20A, Package_SO:SOIC-8_3.9x4.9mm_P1.27mm, F.Cu at (231.1, 82.2)
- added U12: ACS712xLCTR-20A, Package_SO:SOIC-8_3.9x4.9mm_P1.27mm, F.Cu at (231.1, 88.8)
- added U13: ACS712xLCTR-20A, Package_SO:SOIC-8_3.9x4.9mm_P1.27mm, F.Cu at (231.1, 95.4)
- added U15: MIC5219-3.3YM5, Converter_DCDC:Converter_DCDC_Murata_OKI-78SR_Vertical, F.Cu at (245.4, 101.0)
- R5, R7: value R -> 200
Connections:
- J2 pad 1: /OUT_C -> /CON_C
- J2 pad 2: /OUT_B -> /CON_B
- J2 pad 3: /OUT_A -> /CON_A
- R1_T1 pad 2: unconnected-(R1_T1-Pad2) -> /COM
- R1_T1 pad 3: /COM -> unconnected-(R1_T1-Pad3)
